File: OutputStage.sch (KiCad schematic (older format))
At the start: 58 parts, among them Q12 BSC067N06LS3, Q13 BSC067N06LS3, Q3 AON7400A, Q5 AON7400A, U5 LM5175PWPR

Commit message: Much layout. Wow
Parts:
- removed Q3, Q5: AON7400A, lc_lib:QFN-8_3X3X065P, symbol SmartBattery:AO4468
- added Q3, Q5: AON7400A, lc_lib:SON-8_3.3X3.3MM, symbol SmartBattery:AON7400A
Other:
- note added: "CHANGE TO 50V PARTS\n"
Changed lines of the file:
@@
-	1    0    0    -1
-$EndComp
-$Comp
-L SmartBattery:AO4468 Q3
-U 1 1 60419B77
-P 5150 800
-F 0 "Q3" H 5356 846 50  0000 L CNN
-F 1 "AON7400A " H 5356 755 50  0000 L CNN
-F 2 "lc_lib:QFN-8_3X3X065P" H 5350 900 50  0001 C CNN
-F 3 "~" H 5150 800 50  0001 C CNN
-F 4 "AON7400A " H 5150 800 50  0001 C CNN "SKU"
-	1    5150 800
-	1    0    0    -1
-$EndComp
-$Comp
-L SmartBattery:AO4468 Q5
-U 1 1 6041AE7E
-P 5150 1400
-F 0 "Q5" H 5356 1446 50  0000 L CNN
-F 1 "AON7400A " H 5356 1355 50  0000 L CNN
-F 2 "lc_lib:QFN-8_3X3X065P" H 5350 1500 50  0001 C CNN
-F 3 "~" H 5150 1400 50  0001 C CNN
-F 4 "AON7400A " H 5150 1400 50  0001 C CNN "SKU"
-	1    5150 1400
 	1    0    0    -1
 $EndComp
@@
 Text HLabel 8800 1200 3    50   Output ~ 0
 VOLTAGE_CONTROL
+Text Notes 9050 950  0    50   ~ 0
+CHANGE TO 50V PARTS\n
+$Comp
+L SmartBattery:AON7400A Q?
+U 1 1 6008062D
+P 5150 800
+AR Path="/5FD15753/6008062D" Ref="Q?"  Part="1"
+AR Path="/5FD99B08/6008062D" Ref="Q?"  Part="1"
+AR Path="/60413DD6/6008062D" Ref="Q3"  Part="1"
+F 0 "Q3" V 5500 950 50  0000 L CNN
+F 1 "AON7400A" V 5400 750 50  0000 L CNN
+F 2 "lc_lib:SON-8_3.3X3.3MM" H 5800 1250 50  0001 C CNN
+F 3 "~" H 5150 800 50  0001 C CNN
+F 4 "AON7400A" H 5356 755 50  0001 L CNN "SKU"
+F 5 "C85734" H 5356 664 50  0001 L CNN "LCSC"
+	1    5150 800
+	1    0    0    -1
+$EndComp
+$Comp
+L SmartBattery:AON7400A Q?
+U 1 1 60085B05
+P 5150 1400
+AR Path="/5FD15753/60085B05" Ref="Q?"  Part="1"
+AR Path="/5FD99B08/60085B05" Ref="Q?"  Part="1"
+AR Path="/60413DD6/60085B05" Ref="Q5"  Part="1"
+F 0 "Q5" V 5500 1550 50  0000 L CNN
+F 1 "AON7400A" V 5400 1350 50  0000 L CNN
+F 2 "lc_lib:SON-8_3.3X3.3MM" H 5800 1850 50  0001 C CNN
+F 3 "~" H 5150 1400 50  0001 C CNN
+F 4 "AON7400A" H 5356 1355 50  0001 L CNN "SKU"
+F 5 "C85734" H 5356 1264 50  0001 L CNN "LCSC"
+	1    5150 1400
+	1    0    0    -1
+$EndComp
 $EndSCHEMATC
