File: SmartBattery.sch (KiCad schematic (older format))
At the start: 3 parts, among them J1 USB_C_Receptacle_USB2.0, J2 ST-USB-003A, J3 Barrel_Jack_MountingPin

Commit message: Replaced old charger to support JLC assembly. Very close now!
Parts:
- added J15: USB_C_Receptacle_USB2.0, Connector_USB:USB_C_Receptacle_Amphenol_12401548E4-2A, symbol Connector:USB_C_Receptacle_USB2.0
- added J16: Conn_01x03_Female, symbol Connector:Conn_01x03_Female
Connections:
- net labels added: GND
- wire segments 1 -> 20
Other:
- moved on the sheet: J1, J3
Changed lines of the file:
@@
 F2 "BATT_PACK_P" B L 4700 2900 50
 F3 "VSYS" B R 5850 2900 50
-F4 "PMON" I R 5850 3700 50
-F5 "IBAT" I R 5850 3600 50
-F6 "IADP" I R 5850 3500 50
-F7 "ACOK" I R 5850 3400 50
-F8 "PROCHOT_N" I R 5850 3300 50
-F9 "CHARGER_SDA" I R 5850 3200 50
-F10 "CHARGER_SCL" I R 5850 3100 50
-F11 "ADAPTER_IN" I L 4700 3600 50
+F4 "IBAT" I R 5850 3600 50
+F5 "IADP" I R 5850 3500 50
+F6 "PROCHOT_N" I R 5850 3300 50
+F7 "CHARGER_SDA" I R 5850 3200 50
+F8 "CHARGER_SCL" I R 5850 3100 50
+F9 "ADAPTER_IN" I L 4700 3600 50
+F10 "PSYS" I R 5850 3700 50
+F11 "CHRG_OK" I R 5850 3400 50
+F12 "EN_OTG" I L 4700 3450 50
+F13 "BATT_DISCONNECT" B L 4700 3000 50
 $EndSheet
 $Sheet
@@
 L Connector:Barrel_Jack_MountingPin J3
 U 1 1 60145270
-P 3300 4700
-F 0 "J3" H 3357 5017 50  0000 C CNN
-F 1 "Barrel_Jack_MountingPin" H 3357 4926 50  0000 C CNN
-F 2 "Connector_BarrelJack:BarrelJack_Horizontal" H 3350 4660 50  0001 C CNN
-F 3 "~" H 3350 4660 50  0001 C CNN
-F 4 "320120003" H 3300 4700 50  0001 C CNN "SKU"
-	1    3300 4700
+P 3200 4950
+F 0 "J3" H 3257 5267 50  0000 C CNN
+F 1 "Barrel_Jack_MountingPin" H 3257 5176 50  0000 C CNN
+F 2 "Connector_BarrelJack:BarrelJack_Horizontal" H 3250 4910 50  0001 C CNN
+F 3 "~" H 3250 4910 50  0001 C CNN
+F 4 "320120003" H 3200 4950 50  0001 C CNN "SKU"
+	1    3200 4950
 	1    0    0    -1
 $EndComp
 $Sheet
-S 4700 4900 1150 700
+S 7450 1900 1150 700
 U 60413DD6
 F0 "OutputStage" 50
 F1 "OutputStage.sch" 50
+F2 "VSYS" I L 7450 2050 50
+F3 "OUTPUT_VOLTAGE" O R 8600 2050 50
 $EndSheet
 $Sheet
-S 1450 4400 1150 350
+S 7500 2950 1150 350
 U 6041786F
 F0 "Peripheral_3p3v" 50
 F1 "Peripheral_3p3v.sch" 50
+F2 "VSYS" I L 7500 3050 50
+F3 "3p3v" O L 7500 3200 50
 $EndSheet
 $Comp
 L Connector:USB_C_Receptacle_USB2.0 J1
 U 1 1 5FD13F83
-P 1300 1800
-F 0 "J1" H 1407 2667 50  0000 C CNN
-F 1 "USB_C_Receptacle_USB2.0" H 1407 2576 50  0000 C CNN
-F 2 "Connector_USB:USB_C_Receptacle_Amphenol_12401548E4-2A" H 1450 1800 50  0001 C CNN
-F 3 "https://www.usb.org/sites/default/files/documents/usb_type-c.zip" H 1450 1800 50  0001 C CNN
-F 4 "TYPE-C-31-M-17" H 1300 1800 50  0001 C CNN "SKU"
-	1    1300 1800
+P 1200 1450
+F 0 "J1" H 1307 2317 50  0000 C CNN
+F 1 "USB_C_Receptacle_USB2.0" H 1307 2226 50  0000 C CNN
+F 2 "Connector_USB:USB_C_Receptacle_Amphenol_12401548E4-2A" H 1350 1450 50  0001 C CNN
+F 3 "https://www.usb.org/sites/default/files/documents/usb_type-c.zip" H 1350 1450 50  0001 C CNN
+F 4 "TYPE-C-31-M-17" H 1200 1450 50  0001 C CNN "SKU"
+	1    1200 1450
 	1    0    0    -1
 $EndComp
 $Sheet
-S 1700 5300 1400 700
+S 7400 4400 1400 700
 U 5FF1D194
 F0 "MCU" 50
 F1 "MCU.sch" 50
-F2 "Power_3p3v" I L 1700 5400 50
+F2 "Power_3p3v" I L 7400 4500 50
 $EndSheet
+Wire Wire Line
+	6850 2900 6850 3050
+Wire Wire Line
+	6850 3050 7500 3050
+Wire Wire Line
+	5850 2900 6850 2900
+Wire Wire Line
+	7400 4500 6950 4500
+Wire Wire Line
+	6950 4500 6950 3200
+Wire Wire Line
+	6950 3200 7500 3200
+Wire Wire Line
+	6850 2900 6850 2050
+Wire Wire Line
+	6850 2050 7450 2050
+Connection ~ 6850 2900
+Wire Wire Line
+	3500 4850 4250 4850
+Wire Wire Line
+	4250 4850 4250 3600
+Wire Wire Line
+	4250 3600 4700 3600
+$Comp
+L power:GND #PWR0158
+U 1 1 5FFB83C4
+P 3700 5100
+F 0 "#PWR0158" H 3700 4850 50  0001 C CNN
+F 1 "GND" H 3705 4927 50  0000 C CNN
+F 2 "" H 3700 5100 50  0001 C CNN
+F 3 "" H 3700 5100 50  0001 C CNN
+	1    3700 5100
+	1    0    0    -1
+$EndComp
+Wire Wire Line
+	3500 5050 3700 5050
+Wire Wire Line
+	3700 5050 3700 5100
+Wire Wire Line
+	3200 5250 3500 5250
+Wire Wire Line
+	3500 5250 3500 5050
+Connection ~ 3500 5050
+$Comp
+L power:GND #PWR0159
+U 1 1 5FFB939F
+P 7900 1650
+F 0 "#PWR0159" H 7900 1400 50  0001 C CNN
+F 1 "GND" H 8050 1600 50  0000 C CNN
+F 2 "" H 7900 1650 50  0001 C CNN
+F 3 "" H 7900 1650 50  0001 C CNN
+	1    7900 1650
+	1    0    0    -1
+$EndComp
+Wire Wire Line
+	7900 1650 7800 1650
+Connection ~ 7900 1650
+Wire Wire Line
+	9450 2050 9450 1050
+Wire Wire Line
+	9450 1050 8200 1050
+Wire Wire Line
+	8600 2050 9450 2050
+$Comp
+L Connector:USB_C_Receptacle_USB2.0 J15
+U 1 1 60B08C44
+P 2650 1450
+F 0 "J15" H 2757 2317 50  0000 C CNN
+F 1 "USB_C_Receptacle_USB2.0" H 2757 2226 50  0000 C CNN
+F 2 "Connector_USB:USB_C_Receptacle_Amphenol_12401548E4-2A" H 2800 1450 50  0001 C CNN
+F 3 "https://www.usb.org/sites/default/files/documents/usb_type-c.zip" H 2800 1450 50  0001 C CNN
+F 4 "TYPE-C-31-M-17" H 2650 1450 50  0001 C CNN "SKU"
+	1    2650 1450
+	1    0    0    -1
+$EndComp
+$Comp
+L Connector:Conn_01x03_Female J16
+U 1 1 60B1798D
+P 3800 1200
+F 0 "J16" H 3828 1226 50  0000 L CNN
+F 1 "Conn_01x03_Female" H 3828 1135 50  0000 L CNN
+F 2 "" H 3800 1200 50  0001 C CNN
+F 3 "~" H 3800 1200 50  0001 C CNN
+	1    3800 1200
+	1    0    0    -1
+$EndComp
 $EndSCHEMATC

Commit message: Both type-c ports are done! Only outputstage left.
Parts:
- removed J1, J15: USB_C_Receptacle_USB2.0, Connector_USB:USB_C_Receptacle_Amphenol_12401548E4-2A, symbol Connector:USB_C_Receptacle_USB2.0
- added J17, J18: Conn_01x03_Female, symbol Connector:Conn_01x03_Female
- added Q22, Q24: VBA2625, SmartBattery:SOIC127P600X175-8N, symbol SmartBattery:VBA2625
- added Q23: 2n7002K, Package_TO_SOT_SMD:SOT-23, symbol Device:Q_NMOS_GSD
- added R85: 100k, lc_lib:0402_R, symbol Device:R_Small_US
- added U13: TPS2511DGNR, SOP65P490X110-9N, symbol SmartBattery:TPS2511DGNR
Connections:
- wire segments 20 -> 26
Other:
- moved on the sheet: J2
Changed lines of the file:
@@
 $Descr A4 11693 8268
 encoding utf-8
-Sheet 1 6
+Sheet 1 8
 Title ""
 Date ""
@@
 L Connector:USB_B J2
 U 1 1 5FD1640D
-P 7900 1250
-F 0 "J2" H 7957 1717 50  0000 C CNN
-F 1 "ST-USB-003A" H 7957 1626 50  0000 C CNN
-F 2 "Connector_USB:USB3_A_Plug_Wuerth_692112030100_Horizontal" H 8050 1200 50  0001 C CNN
-F 3 " ~" H 8050 1200 50  0001 C CNN
-F 4 "320010007" H 7900 1250 50  0001 C CNN "SKU"
-	1    7900 1250
-	1    0    0    -1
+P 10550 1200
+F 0 "J2" H 10607 1667 50  0000 C CNN
+F 1 "ST-USB-003A" H 10607 1576 50  0000 C CNN
+F 2 "Connector_USB:USB3_A_Plug_Wuerth_692112030100_Horizontal" H 10700 1150 50  0001 C CNN
+F 3 " ~" H 10700 1150 50  0001 C CNN
+F 4 "320010007" H 10550 1200 50  0001 C CNN "SKU"
+	1    10550 1200
+	-1   0    0    1
 $EndComp
 $Sheet
@@
 F3 "3p3v" O L 7500 3200 50
 $EndSheet
-$Comp
-L Connector:USB_C_Receptacle_USB2.0 J1
-U 1 1 5FD13F83
-P 1200 1450
-F 0 "J1" H 1307 2317 50  0000 C CNN
-F 1 "USB_C_Receptacle_USB2.0" H 1307 2226 50  0000 C CNN
-F 2 "Connector_USB:USB_C_Receptacle_Amphenol_12401548E4-2A" H 1350 1450 50  0001 C CNN
-F 3 "https://www.usb.org/sites/default/files/documents/usb_type-c.zip" H 1350 1450 50  0001 C CNN
-F 4 "TYPE-C-31-M-17" H 1200 1450 50  0001 C CNN "SKU"
-	1    1200 1450
-	1    0    0    -1
-$EndComp
-$Sheet
-S 7400 4400 1400 700
+$Sheet
+S 7500 3800 1400 700
 U 5FF1D194
 F0 "MCU" 50
 F1 "MCU.sch" 50
-F2 "Power_3p3v" I L 7400 4500 50
+F2 "Power_3p3v" I L 7500 3900 50
 $EndSheet
 Wire Wire Line
@@
 	5850 2900 6850 2900
 Wire Wire Line
-	7400 4500 6950 4500
-Wire Wire Line
-	6950 4500 6950 3200
+	6950 3950 6950 3900
 Wire Wire Line
 	6950 3200 7500 3200
@@
 	6850 2050 7450 2050
 Connection ~ 6850 2900
-Wire Wire Line
-	3500 4850 4250 4850
-Wire Wire Line
-	4250 4850 4250 3600
-Wire Wire Line
-	4250 3600 4700 3600
 $Comp
 L power:GND #PWR0158
@@
 L power:GND #PWR0159
 U 1 1 5FFB939F
-P 7900 1650
-F 0 "#PWR0159" H 7900 1400 50  0001 C CNN
-F 1 "GND" H 8050 1600 50  0000 C CNN
-F 2 "" H 7900 1650 50  0001 C CNN
-F 3 "" H 7900 1650 50  0001 C CNN
-	1    7900 1650
-	1    0    0    -1
-$EndComp
-Wire Wire Line
-	7900 1650 7800 1650
-Connection ~ 7900 1650
+P 10500 1850
+F 0 "#PWR0159" H 10500 1600 50  0001 C CNN
+F 1 "GND" H 10650 1800 50  0000 C CNN
+F 2 "" H 10500 1850 50  0001 C CNN
+F 3 "" H 10500 1850 50  0001 C CNN
+	1    10500 1850
+	1    0    0    -1
+$EndComp
+Wire Wire Line
+	10500 1850 10400 1850
 Wire Wire Line
 	9450 2050 9450 1050
@@
 	9450 1050 8200 1050
 Wire Wire Line
-	8600 2050 9450 2050
-$Comp
-L Connector:USB_C_Receptacle_USB2.0 J15
-U 1 1 60B08C44
-P 2650 1450
-F 0 "J15" H 2757 2317 50  0000 C CNN
-F 1 "USB_C_Receptacle_USB2.0" H 2757 2226 50  0000 C CNN
-F 2 "Connector_USB:USB_C_Receptacle_Amphenol_12401548E4-2A" H 2800 1450 50  0001 C CNN
-F 3 "https://www.usb.org/sites/default/files/documents/usb_type-c.zip" H 2800 1450 50  0001 C CNN
-F 4 "TYPE-C-31-M-17" H 2650 1450 50  0001 C CNN "SKU"
-	1    2650 1450
-	1    0    0    -1
-$EndComp
+	8600 2050 9000 2050
 $Comp
 L Connector:Conn_01x03_Female J16
 U 1 1 60B1798D
-P 3800 1200
-F 0 "J16" H 3828 1226 50  0000 L CNN
-F 1 "Conn_01x03_Female" H 3828 1135 50  0000 L CNN
-F 2 "" H 3800 1200 50  0001 C CNN
-F 3 "~" H 3800 1200 50  0001 C CNN
-	1    3800 1200
-	1    0    0    -1
-$EndComp
+P 2950 950
+F 0 "J16" H 2978 976 50  0000 L CNN
+F 1 "Conn_01x03_Female" H 2978 885 50  0000 L CNN
+F 2 "" H 2950 950 50  0001 C CNN
+F 3 "~" H 2950 950 50  0001 C CNN
+	1    2950 950
+	1    0    0    -1
+$EndComp
+$Sheet
+S 4600 4200 1900 1050
+U 5FF971C1
+F0 "type_c_input" 50
+F1 "type_c_input.sch" 50
+F2 "INPUT_DM" I R 6500 4250 50
+F3 "INPUT_DP" I R 6500 4350 50
+F4 "INPUT_TYPEC_RST" I R 6500 4500 50
+F5 "INPUT_TYPEC_SDA" I R 6500 4750 50
+F6 "INPUT_TYPEC_SCL" I R 6500 4850 50
+F7 "INPUT_TYPEC_ALERT_N" I R 6500 4950 50
+F8 "INPUT_TYPEC_PWR" I L 4600 4300 50
+F9 "INPUT_TYPEC_VBUS_DIV7" I R 6500 5050 50
+F10 "INPUT_TYPEC_AWAKE" I R 6500 5150 50
+F11 "INPUT_TYPEC_MCUPWR" I R 6500 4600 50
+$EndSheet
+Wire Wire Line
+	6950 3900 7500 3900
+Connection ~ 6950 3900
+Wire Wire Line
+	6950 3900 6950 3200
+$Sheet
+S 9250 2350 1600 1200
+U 600C8F88
+F0 "Type_C_Output" 50
+F1 "Type_C_Output.sch" 50
+F2 "OUTPUT_DM" I R 10850 2400 50
+F3 "OUTPUT_DP" I R 10850 2500 50
+F4 "OUTPUT_TYPEC_SDA" I R 10850 2800 50
+F5 "OUTPUT_TYPEC_SCL" I R 10850 2900 50
+F6 "OUTPUT_TYPEC_ALERT_N" I R 10850 3000 50
+F7 "OUTPUT_TYPEC_VBUS_DIV7" I R 10850 3100 50
+F8 "OUTPUT_TYPEC_PWR" I L 9250 2450 50
+F9 "OUTPUT_TYPEC_MCUPWR" I R 10850 3300 50
+F10 "OUTPUT_TYPEC_RESET" I R 10850 2650 50
+F11 "OUTPUT_TYPEC_VCON" I R 10850 3400 50
+$EndSheet
+Wire Wire Line
+	4250 3600 4700 3600
+Wire Wire Line
+	3500 4850 4250 4850
+Wire Wire Line
+	4250 3600 4250 4300
+Wire Wire Line
+	4250 4300 4600 4300
+Connection ~ 4250 4300
+Wire Wire Line
+	4250 4300 4250 4850
+Wire Wire Line
+	9000 2050 9000 2450
+Wire Wire Line
+	9000 2450 9250 2450
+Connection ~ 9000 2050
+Wire Wire Line
+	9000 2050 9450 2050
+$Comp
+L Connector:Conn_01x03_Female J17
+U 1 1 602EC919
+P 3250 4150
+F 0 "J17" H 3278 4176 50  0000 L CNN
+F 1 "Conn_01x03_Female" H 3278 4085 50  0000 L CNN
+F 2 "" H 3250 4150 50  0001 C CNN
+F 3 "~" H 3250 4150 50  0001 C CNN
+	1    3250 4150
+	-1   0    0    1
+$EndComp
+$Comp
+L Connector:Conn_01x03_Female J18
+U 1 1 602EE89B
+P 4250 900
+F 0 "J18" H 4278 926 50  0000 L CNN
+F 1 "Conn_01x03_Female" H 4278 835 50  0000 L CNN
+F 2 "" H 4250 900 50  0001 C CNN
+F 3 "~" H 4250 900 50  0001 C CNN
+	1    4250 900
+	1    0    0    -1
+$EndComp
+$Comp
+L SmartBattery:TPS2511DGNR U13
+U 1 1 602F0A61
+P 5850 1750
+F 0 "U13" H 5850 2520 50  0000 C CNN
+F 1 "TPS2511DGNR" H 5850 2429 50  0000 C CNN
+F 2 "SOP65P490X110-9N" H 5850 1750 50  0001 L BNN
+F 3 "" H 5850 1750 50  0001 L BNN
+F 4 "C68648" H 5850 1750 50  0001 C CNN "LCSC"
+	1    5850 1750
+	1    0    0    -1
+$EndComp
+$Comp
+L SmartBattery:VBA2625 Q?
+U 1 1 6034999B
+P 2550 5800
+AR Path="/5FF971C1/6034999B" Ref="Q?"  Part="1"
+AR Path="/600C8F88/6034999B" Ref="Q?"  Part="1"
+AR Path="/6034999B" Ref="Q22"  Part="1"
+F 0 "Q22" V 2985 5800 50  0000 C CNN
+F 1 "VBA2625" V 2894 5800 50  0000 C CNN
+F 2 "SmartBattery:SOIC127P600X175-8N" H 2550 5800 50  0001 L BNN
+F 3 "" H 2550 5800 50  0001 L BNN
+F 4 "Alpha & Omega Semiconductor" H 2550 5800 50  0001 L BNN "MANUFACTURER"
+F 5 "I" H 2550 5800 50  0001 L BNN "PARTREV"
+F 6 "IPC 7351B" H 2550 5800 50  0001 L BNN "STANDARD"
+F 7 "1.75 mm" H 2550 5800 50  0001 L BNN "MAXIMUM_PACKAGE_HEIGHT"
+F 8 "C416236" V 2803 5800 50  0000 C CNN "lcsc"
+	1    2550 5800
+	0    1    -1   0
+$EndComp
+$Comp
+L SmartBattery:VBA2625 Q?
+U 1 1 603499A6
+P 3300 5850
+AR Path="/5FF971C1/603499A6" Ref="Q?"  Part="1"
+AR Path="/600C8F88/603499A6" Ref="Q?"  Part="1"
+AR Path="/603499A6" Ref="Q24"  Part="1"
+F 0 "Q24" V 3735 5850 50  0000 C CNN
+F 1 "VBA2625" V 3644 5850 50  0000 C CNN
+F 2 "SmartBattery:SOIC127P600X175-8N" H 3300 5850 50  0001 L BNN
+F 3 "" H 3300 5850 50  0001 L BNN
+F 4 "Alpha & Omega Semiconductor" H 3300 5850 50  0001 L BNN "MANUFACTURER"
+F 5 "I" H 3300 5850 50  0001 L BNN "PARTREV"
+F 6 "IPC 7351B" H 3300 5850 50  0001 L BNN "STANDARD"
+F 7 "1.75 mm" H 3300 5850 50  0001 L BNN "MAXIMUM_PACKAGE_HEIGHT"
+F 8 "C416236" V 3553 5850 50  0000 C CNN "lcsc"
+	1    3300 5850
+	0    -1   -1   0
+$EndComp
+$Comp
+L Device:Q_NMOS_GSD Q?
+U 1 1 603499AC
+P 2850 6450
+AR Path="/5FD15753/603499AC" Ref="Q?"  Part="1"
+AR Path="/600C8F88/603499AC" Ref="Q?"  Part="1"
+AR Path="/603499AC" Ref="Q23"  Part="1"
+F 0 "Q23" H 3055 6404 50  0000 L CNN
+F 1 "2n7002K" H 3055 6495 50  0000 L CNN
+F 2 "Package_TO_SOT_SMD:SOT-23" H 3050 6550 50  0001 C CNN
+F 3 "~" H 2850 6450 50  0001 C CNN
+	1    2850 6450
+	-1   0    0    -1
+$EndComp
+$Comp
+L Device:R_Small_US R?
+U 1 1 603499B3
+P 2950 5850
+AR Path="/5FD99B08/603499B3" Ref="R?"  Part="1"
+AR Path="/5FF1D194/603499B3" Ref="R?"  Part="1"
+AR Path="/5FF971C1/603499B3" Ref="R?"  Part="1"
+AR Path="/600C8F88/603499B3" Ref="R?"  Part="1"
+AR Path="/603499B3" Ref="R85"  Part="1"
+F 0 "R85" V 2900 5700 50  0000 L CNN
+F 1 "100k" V 2900 5950 50  0000 L CNN
+F 2 "lc_lib:0402_R" H 2950 5850 50  0001 C CNN
+F 3 "~" H 2950 5850 50  0001 C CNN
+F 4 "C25741" V 2950 5850 50  0001 C CNN "LCSC"
+	1    2950 5850
+	1    0    0    -1
+$EndComp

Commit message: Added final touches to barrel jack and feedforward.
Need to finish output stage, then add screw terminals.
Parts:
- removed J3: Barrel_Jack_MountingPin, Connector_BarrelJack:BarrelJack_Horizontal, symbol Connector:Barrel_Jack_MountingPin
- removed Q22, Q24: VBA2625, SmartBattery:SOIC127P600X175-8N, symbol SmartBattery:VBA2625
- removed Q23: 2n7002K, Package_TO_SOT_SMD:SOT-23, symbol Device:Q_NMOS_GSD
- removed R85: 100k, lc_lib:0402_R, symbol Device:R_Small_US
- added C112, C113: 10u, lc_lib:0805_C, symbol Device:C_Small
- added D12, D13, D14: B5817W-5819W, lc_lib:SOD-123, symbol Device:D_Small
- added Q22: AO3401A, lc_lib:SOT-23(SOT-23-3), symbol Device:Q_PMOS_GSD
- added U14: HT7533-1, lc_lib:SOT-89(SOT-89-3), symbol SmartBattery:HT7533-1
- U13: footprint SOP65P490X110-9N -> SmartBattery:SOP65P490X110-9N
Connections:
- wire segments 26 -> 22
Changed lines of the file:
@@
 $Descr A4 11693 8268
 encoding utf-8
-Sheet 1 8
+Sheet 1 9
 Title ""
 Date ""
@@
 Wire Wire Line
 	3700 2900 4700 2900
-$Comp
-L Connector:Barrel_Jack_MountingPin J3
-U 1 1 60145270
-P 3200 4950
-F 0 "J3" H 3257 5267 50  0000 C CNN
-F 1 "Barrel_Jack_MountingPin" H 3257 5176 50  0000 C CNN
-F 2 "Connector_BarrelJack:BarrelJack_Horizontal" H 3250 4910 50  0001 C CNN
-F 3 "~" H 3250 4910 50  0001 C CNN
-F 4 "320120003" H 3200 4950 50  0001 C CNN "SKU"
-	1    3200 4950
-	1    0    0    -1
-$EndComp
 $Sheet
 S 7450 1900 1150 700
@@
 	6850 2050 7450 2050
 Connection ~ 6850 2900
-$Comp
-L power:GND #PWR0158
-U 1 1 5FFB83C4
-P 3700 5100
-F 0 "#PWR0158" H 3700 4850 50  0001 C CNN
-F 1 "GND" H 3705 4927 50  0000 C CNN
-F 2 "" H 3700 5100 50  0001 C CNN
-F 3 "" H 3700 5100 50  0001 C CNN
-	1    3700 5100
-	1    0    0    -1
-$EndComp
-Wire Wire Line
-	3500 5050 3700 5050
-Wire Wire Line
-	3700 5050 3700 5100
-Wire Wire Line
-	3200 5250 3500 5250
-Wire Wire Line
-	3500 5250 3500 5050
-Connection ~ 3500 5050
 $Comp
 L power:GND #PWR0159
@@
 F 0 "U13" H 5850 2520 50  0000 C CNN
 F 1 "TPS2511DGNR" H 5850 2429 50  0000 C CNN
-F 2 "SOP65P490X110-9N" H 5850 1750 50  0001 L BNN
+F 2 "SmartBattery:SOP65P490X110-9N" H 5850 1750 50  0001 L BNN
 F 3 "" H 5850 1750 50  0001 L BNN
 F 4 "C68648" H 5850 1750 50  0001 C CNN "LCSC"
@@
 	1    0    0    -1
 $EndComp
-$Comp
-L SmartBattery:VBA2625 Q?
-U 1 1 6034999B
-P 2550 5800
-AR Path="/5FF971C1/6034999B" Ref="Q?"  Part="1"
-AR Path="/600C8F88/6034999B" Ref="Q?"  Part="1"
-AR Path="/6034999B" Ref="Q22"  Part="1"
-F 0 "Q22" V 2985 5800 50  0000 C CNN
-F 1 "VBA2625" V 2894 5800 50  0000 C CNN
-F 2 "SmartBattery:SOIC127P600X175-8N" H 2550 5800 50  0001 L BNN
-F 3 "" H 2550 5800 50  0001 L BNN
-F 4 "Alpha & Omega Semiconductor" H 2550 5800 50  0001 L BNN "MANUFACTURER"
-F 5 "I" H 2550 5800 50  0001 L BNN "PARTREV"
-F 6 "IPC 7351B" H 2550 5800 50  0001 L BNN "STANDARD"
-F 7 "1.75 mm" H 2550 5800 50  0001 L BNN "MAXIMUM_PACKAGE_HEIGHT"
-F 8 "C416236" V 2803 5800 50  0000 C CNN "lcsc"
-	1    2550 5800
-	0    1    -1   0
-$EndComp
-$Comp
-L SmartBattery:VBA2625 Q?
-U 1 1 603499A6
-P 3300 5850
-AR Path="/5FF971C1/603499A6" Ref="Q?"  Part="1"
-AR Path="/600C8F88/603499A6" Ref="Q?"  Part="1"
-AR Path="/603499A6" Ref="Q24"  Part="1"
-F 0 "Q24" V 3735 5850 50  0000 C CNN
-F 1 "VBA2625" V 3644 5850 50  0000 C CNN
-F 2 "SmartBattery:SOIC127P600X175-8N" H 3300 5850 50  0001 L BNN
-F 3 "" H 3300 5850 50  0001 L BNN
-F 4 "Alpha & Omega Semiconductor" H 3300 5850 50  0001 L BNN "MANUFACTURER"
-F 5 "I" H 3300 5850 50  0001 L BNN "PARTREV"
-F 6 "IPC 7351B" H 3300 5850 50  0001 L BNN "STANDARD"
-F 7 "1.75 mm" H 3300 5850 50  0001 L BNN "MAXIMUM_PACKAGE_HEIGHT"
-F 8 "C416236" V 3553 5850 50  0000 C CNN "lcsc"
-	1    3300 5850
-	0    -1   -1   0
-$EndComp
-$Comp
-L Device:Q_NMOS_GSD Q?
-U 1 1 603499AC
-P 2850 6450
-AR Path="/5FD15753/603499AC" Ref="Q?"  Part="1"
-AR Path="/600C8F88/603499AC" Ref="Q?"  Part="1"
-AR Path="/603499AC" Ref="Q23"  Part="1"
-F 0 "Q23" H 3055 6404 50  0000 L CNN
-F 1 "2n7002K" H 3055 6495 50  0000 L CNN
-F 2 "Package_TO_SOT_SMD:SOT-23" H 3050 6550 50  0001 C CNN
-F 3 "~" H 2850 6450 50  0001 C CNN
-	1    2850 6450
-	-1   0    0    -1
-$EndComp
-$Comp
-L Device:R_Small_US R?
-U 1 1 603499B3
-P 2950 5850
-AR Path="/5FD99B08/603499B3" Ref="R?"  Part="1"
-AR Path="/5FF1D194/603499B3" Ref="R?"  Part="1"
-AR Path="/5FF971C1/603499B3" Ref="R?"  Part="1"
-AR Path="/600C8F88/603499B3" Ref="R?"  Part="1"
-AR Path="/603499B3" Ref="R85"  Part="1"
-F 0 "R85" V 2900 5700 50  0000 L CNN
-F 1 "100k" V 2900 5950 50  0000 L CNN
-F 2 "lc_lib:0402_R" H 2950 5850 50  0001 C CNN
-F 3 "~" H 2950 5850 50  0001 C CNN
-F 4 "C25741" V 2950 5850 50  0001 C CNN "LCSC"
-	1    2950 5850
-	1    0    0    -1
+$Sheet
+S 2400 4750 1100 650
+U 5FF4A13F
+F0 "Barrel_Jack_Input" 50
+F1 "Barrel_Jack_Input.sch" 50
+F2 "BARREL_OUTPUT_V" I R 3500 4850 50
+F3 "BARREL_ENABLE" I R 3500 5100 50
+F4 "BARREL_RAW" I R 3500 5250 50
+$EndSheet
+$Comp
+L SmartBattery:HT7533-1 U14
+U 1 1 5FF9C977
+P 8350 5800
+F 0 "U14" H 8325 6315 50  0000 C CNN
+F 1 "HT7533-1" H 8325 6224 50  0000 C CNN
+F 2 "lc_lib:SOT-89(SOT-89-3)" H 8350 5850 50  0001 C CNN
+F 3 "" H 8350 5850 50  0001 C CNN
+F 4 "C14289" H 8325 6133 50  0000 C CNN "LCSC"
+	1    8350 5800
+	1    0    0    -1
+$EndComp
+$Comp
+L Device:D_Small D?
+U 1 1 5FF9C97E
+P 7650 5900
+AR Path="/5FD99B08/5FF9C97E" Ref="D?"  Part="1"
+AR Path="/6041786F/5FF9C97E" Ref="D?"  Part="1"
+AR Path="/5FF9C97E" Ref="D12"  Part="1"
+F 0 "D12" H 7650 6105 50  0000 C CNN
+F 1 "B5817W-5819W" H 7650 6014 50  0000 C CNN
+F 2 "lc_lib:SOD-123" V 7650 5900 50  0001 C CNN
+F 3 "~" V 7650 5900 50  0001 C CNN
+F 4 "304040005" H 7650 5900 50  0001 C CNN "lcsc"
+	1    7650 5900
+	0    1    1    0
+$EndComp
+$Comp
+L Device:D_Small D?
+U 1 1 5FF9C985
+P 9300 5750
+AR Path="/5FD99B08/5FF9C985" Ref="D?"  Part="1"
+AR Path="/6041786F/5FF9C985" Ref="D?"  Part="1"
+AR Path="/5FF9C985" Ref="D13"  Part="1"
+F 0 "D13" H 9300 5955 50  0000 C CNN
+F 1 "B5817W-5819W" H 9300 5864 50  0000 C CNN
+F 2 "lc_lib:SOD-123" V 9300 5750 50  0001 C CNN
+F 3 "~" V 9300 5750 50  0001 C CNN
+F 4 "304040005" H 9300 5750 50  0001 C CNN "lcsc"
+	1    9300 5750
+	0    1    1    0
+$EndComp
+$Comp
+L Device:D_Small D?
+U 1 1 5FF9C98C
+P 9600 5750
+AR Path="/5FD99B08/5FF9C98C" Ref="D?"  Part="1"
+AR Path="/6041786F/5FF9C98C" Ref="D?"  Part="1"
+AR Path="/5FF9C98C" Ref="D14"  Part="1"
+F 0 "D14" H 9600 5955 50  0000 C CNN
+F 1 "B5817W-5819W" H 9600 5864 50  0000 C CNN
+F 2 "lc_lib:SOD-123" V 9600 5750 50  0001 C CNN
+F 3 "~" V 9600 5750 50  0001 C CNN
+F 4 "304040005" H 9600 5750 50  0001 C CNN "lcsc"
+	1    9600 5750
+	0    1    1    0
+$EndComp
+$Comp
+L Device:Q_PMOS_GSD Q22
+U 1 1 5FF9C993
+P 10300 5300
+F 0 "Q22" H 10506 5346 50  0000 L CNN
+F 1 "AO3401A" H 10506 5255 50  0000 L CNN
+F 2 "lc_lib:SOT-23(SOT-23-3)" H 10500 5400 50  0001 C CNN
+F 3 "~" H 10300 5300 50  0001 C CNN
+F 4 "C15127" H 10300 5300 50  0001 C CNN "LCSC"
+	1    10300 5300
+	1    0    0    -1
+$EndComp
+$Comp
+L Device:C_Small C?
+U 1 1 5FF9C99A
+P 10200 5950
+AR Path="/5FD99B08/5FF9C99A" Ref="C?"  Part="1"
+AR Path="/6041786F/5FF9C99A" Ref="C?"  Part="1"
+AR Path="/5FF9C99A" Ref="C112"  Part="1"
+F 0 "C112" H 10292 5996 50  0000 L CNN
+F 1 "10u" H 10292 5905 50  0000 L CNN
+F 2 "lc_lib:0805_C" H 10200 5950 50  0001 C CNN
+F 3 "~" H 10200 5950 50  0001 C CNN
+F 4 "C15850" H 10200 5950 50  0001 C CNN "LCSC"
+	1    10200 5950
+	-1   0    0    1
+$EndComp
+$Comp
+L Device:C_Small C?
+U 1 1 5FF9C9A1
+P 10550 5950
+AR Path="/5FD99B08/5FF9C9A1" Ref="C?"  Part="1"
+AR Path="/6041786F/5FF9C9A1" Ref="C?"  Part="1"
+AR Path="/5FF9C9A1" Ref="C113"  Part="1"
+F 0 "C113" H 10642 5996 50  0000 L CNN
+F 1 "10u" H 10642 5905 50  0000 L CNN
+F 2 "lc_lib:0805_C" H 10550 5950 50  0001 C CNN
+F 3 "~" H 10550 5950 50  0001 C CNN
+F 4 "C15850" H 10550 5950 50  0001 C CNN "LCSC"
+	1    10550 5950
+	-1   0    0    1
 $EndComp
 $EndSCHEMATC
